File: badge.brd (EAGLE design)
At the start: 91 x 92.5 mm, 177 parts, among them CN4 MicroUSB, IC3 MEGA8-AI, Q1 BSS138, Q2 BSS138, T1 MMUN2133LT1G, U1 TPS61090RSAR, U2 MCP73871, U3 LIS3DHTR, U4 MIC5225-3.3, Y1 16.00MHz

Commit message: ready for production
Parts:
- removed BT1: (no value), SparkFun-Batteries:BATTERY_18650-HOLDER
- removed S1: (no value), adafruit:EG1218
- added U$17: CL-SB-12A-02T, defcon:CL-SB-12A-02T
- added U$22: 54_BATTERY_CLIP, defcon:54_BATTERY_CLIP
- C6: value 100uF -> 10uF
Connections:
- net BOOST_ENABLE: now also U$17.P$2; no longer S1.P
- net GND: now also U$17.P$3, U$22.P$4, U$22.P$5, U$22.P$6; no longer BT1.GND@1, S1.S
- net VLIPO: now also U$22.P$1, U$22.P$2, U$22.P$3; no longer BT1.PWR@1
Routing:
- net VLIPO: track 59.1 -> 78.9 mm
- net BOOST_ENABLE: track 43.0 -> 45.0 mm, vias 1 -> 2
Other:
- board text added: "0x4d 0x63 0x41 0x66 0x65 0x65 0x20 0x4c 0x69 0x76 0x65 0x73"
- board text added: "ON"
Changed lines of the file:
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@@
 <setting verticaltext="up"/>
 </settings>
-<grid distance="0.1" unitdist="mm" unit="mm" style="lines" multiple="1" display="yes" altdistance="5" altunitdist="mil" altunit="mil"/>
+<grid distance="1" unitdist="mil" unit="mil" style="lines" multiple="1" display="yes" altdistance="5" altunitdist="mil" altunit="mil"/>
 <layers>
 <layer number="1" name="Top" color="4" fill="1" visible="yes" active="yes"/>
@@
 <dimension x1="0" y1="0" x2="100" y2="0" x3="50" y3="-6" textsize="1.778" layer="51"/>
 <dimension x1="100" y1="0" x2="100" y2="100" x3="105.5" y3="50" textsize="1.778" layer="51"/>
-<text x="50.861821875" y="72.62003125" size="1.778" layer="30" font="vector" ratio="20" rot="MR0">fir3r007
+<text x="50.861821875" y="73.12803125" size="1.778" layer="30" font="vector" ratio="20" rot="MR0">fir3r007
 ichorous
 videlen</text>
@@
 <vertex x="68.007765625" y="83.002390625"/>
 </polygon>
+<text x="54.0004" y="3.0734" size="1.4224" layer="25" font="vector" ratio="20" rot="MR0">ON</text>
+<text x="65.278" y="67.2338" size="1.778" layer="16" font="vector" ratio="20" rot="MR0">0x4d 0x63 0x41 0x66 0x65 0x65
+0x20 0x4c 0x69 0x76 0x65 0x73</text>
 </plain>
 <attributes>
@@
 </element>
 <element name="T1" library="piboy_new" package="TRANSISTOR_SC59-BEC" value="MMUN2133LT1G" x="23.17670625" y="15.568790625" rot="MR270"/>
-<element name="C6" library="resistor" library_urn="urn:adsk.eagle:library:348" package="C1210" package3d_urn="urn:adsk.eagle:package:26139/1" value="100uF" x="41.558" y="12.5184" smashed="yes" rot="MR180">
+<element name="C6" library="resistor" library_urn="urn:adsk.eagle:library:348" package="C1210" package3d_urn="urn:adsk.eagle:package:26139/1" value="10uF" x="41.558" y="12.5184" smashed="yes" rot="MR180">
 <attribute name="NAME" x="44.0175125" y="14.126434375" size="0.6096" layer="26" font="vector" ratio="20" rot="MR0"/>
 </element>
@@
 <attribute name="NAME" x="45.5841" y="9.07415" size="0.6096" layer="26" font="vector" ratio="20" rot="MR270"/>
 </element>
-<element name="BT1" library="SparkFun-Batteries" package="BATTERY_18650-HOLDER" value="" x="45.0502" y="26.3206" rot="MR0">
-<attribute name="PROD_ID" value="BATT-12327" x="45.0502" y="26.3206" size="1.778" layer="28" rot="MR0" display="off"/>
-<attribute name="SF_SKU" value="PRT-13113" x="45.0502" y="26.3206" size="1.778" layer="28" rot="MR0" display="off"/>
-</element>
 <element name="IC3" library="atmel" library_urn="urn:adsk.eagle:library:105" package="TQFP32-08" package3d_urn="urn:adsk.eagle:package:4313/1" value="MEGA8-AI" x="39.05088125" y="26.360534375" smashed="yes" rot="R45">
 <attribute name="MF" value="" x="39.05088125" y="26.360534375" size="1.778" layer="27" rot="R45" display="off"/>
@@
 <attribute name="NAME" x="74.675271875" y="73.097371875" size="0.6096" layer="26" font="vector" ratio="20" rot="MR180"/>
 </element>
-<element name="S1" library="adafruit" library_urn="urn:adsk.eagle:library:420" package="EG1218" value="" x="58" y="6" smashed="yes" rot="R206.5"/>
 <element name="STAT1" library="piboy_new" package="ADAFRUIT_CHIPLED_0603" value="GREEN" x="27" y="29.5" rot="R90"/>
 <element name="STAT2" library="piboy_new" package="ADAFRUIT_CHIPLED_0603" value="GREEN" x="27" y="27.5" rot="R90"/>
@@
 </element>
 <element name="JP3" library="pinhead" library_urn="urn:adsk.eagle:library:325" package="2X04" package3d_urn="urn:adsk.eagle:package:22461/2" value="TCVR_HEADER" x="21" y="77" smashed="yes" rot="R39.3"/>
+<element name="U$17" library="defcon" package="CL-SB-12A-02T" value="CL-SB-12A-02T" x="58.9576" y="6.2984" rot="MR160.8"/>
+<element name="U$22" library="defcon" package="54_BATTERY_CLIP" value="54_BATTERY_CLIP" x="45.8194" y="25.7834" rot="R180"/>
 </elements>
 <signals>
@@
 <contactref element="U2" pad="P$21"/>
 <contactref element="THERM" pad="1"/>
-<contactref element="BT1" pad="GND@1"/>
 <contactref element="IC3" pad="3"/>
 <contactref element="IC3" pad="5"/>
@@
 <contactref element="SW5" pad="P$1"/>
 <contactref element="SW6" pad="P$1"/>
-<contactref element="S1" pad="S"/>
 <contactref element="R21" pad="1"/>
 <contactref element="R22" pad="1"/>
@@
 <wire x1="49.252634375" y1="25.9846875" x2="49.252634375" y2="26.248896875" width="0.3048" layer="1"/>
 <wire x1="49.252634375" y1="26.248896875" x2="48.81415" y2="26.68738125" width="0.3048" layer="1"/>
+<contactref element="U$17" pad="P$3"/>
+<contactref element="U$22" pad="P$4"/>
+<contactref element="U$22" pad="P$5"/>
+<contactref element="U$22" pad="P$6"/>
 </signal>
 <signal name="N$1">
@@
 <contactref element="U1" pad="11"/>
 <contactref element="R13" pad="2"/>
-<contactref element="S1" pad="P"/>
 <wire x1="33.3792" y1="13.0194" x2="31.324478125" y2="13.0194" width="0.3048" layer="16"/>
 <wire x1="31.324478125" y1="13.0194" x2="30.90115625" y2="13.442721875" width="0.3048" layer="16"/>
 <wire x1="40.55180625" y1="15.54048125" x2="40.55180625" y2="15.5404875" width="0.3048" layer="1"/>
-<wire x1="56.98306875" y1="15.4459375" x2="56.4282625" y2="16.00074375" width="0.3048" layer="1"/>
 <wire x1="48.110040625" y1="16.00074375" x2="56.4282625" y2="16.00074375" width="0.3048" layer="1"/>
 <wire x1="40.55180625" y1="15.5404875" x2="41.0120625" y2="16.00074375" width="0.3048" layer="1"/>
-<wire x1="56.98306875" y1="8.806496875" x2="56.98306875" y2="15.4459375" width="0.3048" layer="1"/>
 <wire x1="36.71455" y1="10.9848" x2="37.1888" y2="11.45905" width="0.3048" layer="1"/>
 <wire x1="33.359078125" y1="10.9848" x2="30.90115625" y2="13.442721875" width="0.3048" layer="1"/>
@@
 <wire x1="44.864090625" y1="16.82185625" x2="47.288928125" y2="16.82185625" width="0.3048" layer="1"/>
 <wire x1="47.288928125" y1="16.82185625" x2="48.110040625" y2="16.00074375" width="0.3048" layer="1"/>
-<wire x1="58" y1="6" x2="58" y2="7.789565625" width="0.3048" layer="1"/>
-<wire x1="58" y1="7.789565625" x2="56.98306875" y2="8.806496875" width="0.3048" layer="1"/>
+<wire x1="56.4282625" y1="16.00074375" x2="56.98306875" y2="15.4459375" width="0.3048" layer="1"/>
+<wire x1="56.98306875" y1="15.4459375" x2="56.98306875" y2="11.989765625" width="0.3048" layer="1"/>
+<contactref element="U$17" pad="P$2"/>
+<wire x1="56.98306875" y1="11.989765625" x2="57.022034375" y2="11.989765625" width="0.3048" layer="1"/>
+<wire x1="57.022034375" y1="11.989765625" x2="58.4708" y2="10.541" width="0.3048" layer="1"/>
+<wire x1="58.4708" y1="10.541" x2="58.4708" y2="5.873559375" width="0.3048" layer="1"/>
+<wire x1="58.4708" y1="5.873559375" x2="59.5495625" y2="4.598521875" width="0.3048" layer="16"/>
+<via x="58.4708" y="5.873559375" extent="1-16" drill="0.35"/>
 </signal>
 <signal name="N$5">
@@
 <contactref element="U2" pad="P$15"/>
 <contactref element="U2" pad="P$16"/>
-<contactref element="BT1" pad="PWR@1"/>
 <wire x1="51.3994" y1="15.6166" x2="51.318696875" y2="15.535896875" width="0.3048" layer="16"/>
 <wire x1="50.4344" y1="14.6516" x2="50.4344" y2="14.3539625" width="0.3048" layer="16"/>
@@
 <wire x1="64.906925" y1="30.699284375" x2="64.896078125" y2="30.71013125" width="1.016" layer="16"/>
 <via x="64.906925" y="30.699284375" extent="1-16" drill="0.35" diameter="1.05"/>
-<wire x1="75.6782" y1="26.3106" x2="71.0554" y2="30.9334" width="1.016" layer="1"/>
-<wire x1="75.6782" y1="26.3106" x2="75.6782" y2="26.3478" width="1.016" layer="1"/>
-<wire x1="75.6782" y1="26.3478" x2="81.0378" y2="31.7074" width="1.016" layer="1"/>
 <via x="81.0378" y="31.7074" extent="1-16" drill="0.35" diameter="1.05"/>
-<wire x1="65.141040625" y1="30.9334" x2="64.906925" y2="30.699284375" width="1.016" layer="1"/>
-<wire x1="71.0554" y1="30.9334" x2="65.141040625" y2="30.9334" width="1.016" layer="1"/>
+<wire x1="64.906925" y1="30.699284375" x2="65.141040625" y2="30.9334" width="1.016" layer="1"/>
+<wire x1="65.141040625" y1="30.9334" x2="71.0554" y2="30.9334" width="1.016" layer="1"/>
 <wire x1="51.318696875" y1="15.535896875" x2="51.311946875" y2="15.535896875" width="0.4064" layer="16"/>
 <wire x1="51.311946875" y1="15.535896875" x2="50.517390625" y2="16.330453125" width="0.4064" layer="16"/>
@@
 <wire x1="49.77943125" y1="16.213153125" x2="49.77943125" y2="15.584684375" width="0.6096" layer="16"/>
 <wire x1="49.47049375" y1="15.275746875" x2="49.77943125" y2="15.584684375" width="0.6096" layer="16"/>
+<contactref element="U$22" pad="P$1"/>
+<contactref element="U$22" pad="P$2"/>
+<contactref element="U$22" pad="P$3"/>
+<wire x1="72.393875" y1="25.0474875" x2="71.6234875" y2="25.0474875" width="1.016" layer="1"/>
+<wire x1="71.6234875" y1="25.0474875" x2="69.8194" y2="23.2434" width="1.016" layer="1"/>
+<wire x1="73.1297875" y1="25.7834" x2="77.4394" y2="25.7834" width="1.016" layer="1"/>
+<wire x1="73.1297875" y1="25.7834" x2="72.393875" y2="25.0474875" width="1.016" layer="1"/>
+<wire x1="69.8194" y1="23.2434" x2="69.8194" y2="28.3234" width="1.016" layer="1"/>
+<wire x1="69.8194" y1="28.3234" x2="69.8194" y2="29.6974" width="1.016" layer="1"/>
+<wire x1="69.8194" y1="29.6974" x2="71.0554" y2="30.9334" width="1.016" layer="1"/>
+<wire x1="71.0554" y1="30.9334" x2="72.2894" y2="30.9334" width="1.016" layer="1"/>
+<wire x1="72.2894" y1="30.9334" x2="77.4394" y2="25.7834" width="1.016" layer="1"/>
+<wire x1="77.4394" y1="25.7834" x2="76.2426" y2="25.7834" width="1.016" layer="1"/>
+<wire x1="77.4394" y1="25.7834" x2="77.4394" y2="28.109" width="1.016" layer="1"/>
+<wire x1="77.4394" y1="28.109" x2="81.0378" y2="31.7074" width="1.016" layer="1"/>
 </signal>
 <signal name="N$8">
