File: badge.sch (EAGLE design)
At the start: 177 parts, among them CN4 MicroUSB, IC3 MEGA8-AI, Q1 BSS138, Q2 BSS138, T1 MMUN2133LT1G, U1 TPS61090RSAR, U2 MCP73871, U3 LIS3DHTR, U4 MIC5225-3.3, Y1 16.00MHz

Commit message: ready for production
Parts:
- removed BT1: (no value), SparkFun-Batteries:BATTERY-18650
- removed S1: (no value), adafruit:EG1218S
- added U$17: CL-SB-12A-02T, defcon:CL-SB-12A-02T
- added U$22: 54_BATTERY_CLIP, defcon:54_BATTERY_CLIP
- C6: value 100uF -> 10uF
Connections:
- net BOOST_ENABLE: now also U$17.P$2; no longer S1.P
- net GND: now also U$17.P$3, U$22.P$2; no longer BT1.-, S1.S
- net VLIPO: now also U$22.P$1; no longer BT1.+
Changed lines of the file:
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@@
 <part name="U$23" library="microbuilder" deviceset="VBAT" device=""/>
 <part name="T1" library="piboy_new" deviceset="TRANSISTOR_*-PNP_DRIVER-" device="SC59-BEC" technology="MUN2113T1" value="MMUN2133LT1G"/>
-<part name="C6" library="resistor" library_urn="urn:adsk.eagle:library:348" deviceset="C-US" device="C1210" package3d_urn="urn:adsk.eagle:package:26139/1" value="100uF"/>
+<part name="C6" library="resistor" library_urn="urn:adsk.eagle:library:348" deviceset="C-US" device="C1210" package3d_urn="urn:adsk.eagle:package:26139/1" value="10uF"/>
 <part name="P+1" library="supply1" library_urn="urn:adsk.eagle:library:371" deviceset="+5V" device=""/>
-<part name="U$5" library="microbuilder" deviceset="GND" device=""/>
 <part name="GND1" library="supply1" deviceset="GND" device=""/>
 <part name="R6" library="adafruit" deviceset="R-US_" device="R0805" value="270K"/>
@@
 <part name="U2" library="microbuilder" deviceset="MCP73871" device="" value="MCP73871"/>
 <part name="C8" library="adafruit" deviceset="C-US" device="C0805" value="10uf"/>
-<part name="BT1" library="SparkFun-Batteries" deviceset="BATTERY" device="-18650"/>
 <part name="IC3" library="atmel" library_urn="urn:adsk.eagle:library:105" deviceset="MEGA8" device="-AI" package3d_urn="urn:adsk.eagle:package:4313/1"/>
 <part name="C3" library="resistor" library_urn="urn:adsk.eagle:library:348" deviceset="C-US" device="C0603" package3d_urn="urn:adsk.eagle:package:26138/1" value="22pF"/>
@@
 <part name="GND18" library="supply1" library_urn="urn:adsk.eagle:library:371" deviceset="GND" device=""/>
 <part name="GND19" library="supply1" library_urn="urn:adsk.eagle:library:371" deviceset="GND" device=""/>
-<part name="S1" library="adafruit" library_urn="urn:adsk.eagle:library:420" deviceset="EG1218" device="S"/>
-<part name="U$22" library="microbuilder" deviceset="GND" device=""/>
 <part name="STAT1" library="piboy_new" deviceset="ADAFRUIT_LED" device="CHIPLED_0603" value="GREEN"/>
 <part name="STAT2" library="piboy_new" deviceset="ADAFRUIT_LED" device="CHIPLED_0603" value="GREEN"/>
@@
 <part name="P+4" library="supply1" library_urn="urn:adsk.eagle:library:371" deviceset="+5V" device=""/>
 <part name="P+5" library="supply1" library_urn="urn:adsk.eagle:library:371" deviceset="+5V" device=""/>
+<part name="U$17" library="defcon" deviceset="CL-SB-12A-02T" device=""/>
+<part name="U$25" library="microbuilder" deviceset="GND" device=""/>
+<part name="U$22" library="defcon" deviceset="54_BATTERY_CLIP" device=""/>
+<part name="GND8" library="supply1" deviceset="GND" device=""/>
 </parts>
 <sheets>
@@
 <instance part="C6" gate="G$1" x="-68.58" y="-2.54"/>
 <instance part="P+1" gate="1" x="-45.72" y="0" rot="R270"/>
-<instance part="U$5" gate="G$1" x="-22.86" y="-119.38"/>
 <instance part="GND1" gate="1" x="-55.88" y="-104.14" rot="R90"/>
 <instance part="R6" gate="G$1" x="-106.68" y="-58.42" rot="R90"/>
@@
 <instance part="U2" gate="G$1" x="-78.74" y="-88.9"/>
 <instance part="C8" gate="G$1" x="-116.84" y="-144.78"/>
-<instance part="BT1" gate="G$1" x="-22.86" y="-101.6" rot="R270"/>
 <instance part="IC3" gate="G$1" x="-218.44" y="-2.54"/>
 <instance part="C3" gate="G$1" x="-254" y="-2.54" rot="R270"/>
@@
 <instance part="GND18" gate="1" x="-266.7" y="-93.98" rot="R270"/>
 <instance part="GND19" gate="1" x="-220.98" y="-93.98" rot="R270"/>
-<instance part="S1" gate="1" x="-30.48" y="-7.62" rot="R270"/>
-<instance part="U$22" gate="G$1" x="-22.86" y="-15.24"/>
 <instance part="STAT1" gate="G$1" x="-261.62" y="-121.92" rot="R90"/>
 <instance part="STAT2" gate="G$1" x="-261.62" y="-137.16" rot="R90"/>
@@
 <instance part="P+4" gate="1" x="-378.46" y="12.7"/>
 <instance part="P+5" gate="1" x="-370.84" y="-30.48"/>
+<instance part="U$17" gate="G$1" x="-27.94" y="-7.62"/>
+<instance part="U$25" gate="G$1" x="-20.32" y="-25.4"/>
+<instance part="U$22" gate="G$1" x="-22.86" y="-104.14"/>
+<instance part="GND8" gate="1" x="-22.86" y="-129.54"/>
 </instances>
 <busses>
@@
 </segment>
 <segment>
-<pinref part="BT1" gate="G$1" pin="-"/>
-<pinref part="U$5" gate="G$1" pin="GND"/>
-<wire x1="-22.86" y1="-106.68" x2="-22.86" y2="-116.84" width="0.1524" layer="91"/>
-</segment>
-<segment>
 <pinref part="IC3" gate="G$1" pin="GND"/>
 <pinref part="GND3" gate="1" pin="GND"/>
@@
 <pinref part="GND19" gate="1" pin="GND"/>
 <wire x1="-215.9" y1="-93.98" x2="-218.44" y2="-93.98" width="0.1524" layer="91"/>
-</segment>
-<segment>
-<pinref part="S1" gate="1" pin="S"/>
-<wire x1="-25.4" y1="-12.7" x2="-22.86" y2="-12.7" width="0.1524" layer="91"/>
-<pinref part="U$22" gate="G$1" pin="GND"/>
 </segment>
 <segment>
@@
 <pinref part="GND7" gate="1" pin="GND"/>
 <wire x1="312.42" y1="-111.76" x2="312.42" y2="-116.84" width="0.1524" layer="91"/>
+<junction x="-2.54" y="-27.94"/>
 </segment>
 <segment>
@@
 <pinref part="GND29" gate="1" pin="GND"/>
 <wire x1="-190.5" y1="-101.6" x2="-190.5" y2="-104.14" width="0.1524" layer="91"/>
+</segment>
+<segment>
+<pinref part="U$17" gate="G$1" pin="P$3"/>
+<pinref part="U$25" gate="G$1" pin="GND"/>
+<wire x1="-20.32" y1="-10.16" x2="-20.32" y2="-22.86" width="0.1524" layer="91"/>
+</segment>
+<segment>
+<pinref part="U$22" gate="G$1" pin="P$2"/>
+<wire x1="-22.86" y1="-111.76" x2="-22.86" y2="-127" width="0.1524" layer="91"/>
+<pinref part="GND8" gate="1" pin="GND"/>
 </segment>
 </net>
@@
 </segment>
 <segment>
-<pinref part="S1" gate="1" pin="P"/>
-<wire x1="-35.56" y1="-10.16" x2="-40.64" y2="-10.16" width="0.1524" layer="91"/>
-<label x="-40.64" y="-10.16" size="1.778" layer="95" rot="R270"/>
+<label x="-27.94" y="-25.4" size="1.778" layer="95" rot="R270"/>
+<pinref part="U$17" gate="G$1" pin="P$2"/>
+<wire x1="-27.94" y1="-25.4" x2="-27.94" y2="-10.16" width="0.1524" layer="91"/>
 </segment>
 </net>
@@
 <junction x="-60.96" y="-86.36"/>
 <label x="-33.02" y="-86.36" size="1.778" layer="95"/>
-<pinref part="BT1" gate="G$1" pin="+"/>
 <wire x1="-40.64" y1="-86.36" x2="-22.86" y2="-86.36" width="0.1524" layer="91"/>
-<wire x1="-22.86" y1="-86.36" x2="-22.86" y2="-96.52" width="0.1524" layer="91"/>
-</segment>
-</net>
+<wire x1="-22.86" y1="-86.36" x2="-22.86" y2="-99.06" width="0.1524" layer="91"/>
+<pinref part="U$22" gate="G$1" pin="P$1"/>
+</segment>
+</net>
